Commit message: Update EgoMimic training, evaluation, and calibration code

File: egomimic/resources/model.urdf (robot description, URDF)
Before this commit: robot vx300s, 14 links, 13 joints
Links:
- removed link vx300s/base_link
- removed link vx300s/ee_arm_link
- removed link vx300s/ee_gripper_link
- removed link vx300s/fingers_link
- removed link vx300s/gripper_bar_link
- removed link vx300s/gripper_link
- removed link vx300s/gripper_prop_link
- removed link vx300s/left_finger_link
- removed link vx300s/lower_forearm_link
- removed link vx300s/right_finger_link
- removed link vx300s/shoulder_link
- removed link vx300s/upper_arm_link
- removed link vx300s/upper_forearm_link
- removed link vx300s/wrist_link
- added link base_link, mass 1.02; collision mesh filename=meshes/base_link.STL; visual mesh filename=meshes/base_link.STL
- added link dummy_link
- added link gripper_base, mass 0.45; collision mesh filename=meshes/gripper_base.STL; visual mesh filename=meshes/gripper_base.STL
- added link link1, mass 0.71; collision mesh filename=meshes/link1.STL; visual mesh filename=meshes/link1.STL
- added link link2, mass 1.17; collision mesh filename=meshes/link2.STL; visual mesh filename=meshes/link2.STL
- added link link3, mass 0.5; collision mesh filename=meshes/link3.STL; visual mesh filename=meshes/link3.STL
- added link link4, mass 0.38; collision mesh filename=meshes/link4.STL; visual mesh filename=meshes/link4.STL
- added link link5, mass 0.383; collision mesh filename=meshes/link5.STL; visual mesh filename=meshes/link5.STL
- added link link6, mass 0.00699089613564366; collision mesh filename=meshes/link6.STL; visual mesh filename=meshes/link6.STL
- added link link7, mass 0.025; collision mesh filename=meshes/link7.STL; visual mesh filename=meshes/link7.STL
- added link link8, mass 0.025; collision mesh filename=meshes/link8.STL; visual mesh filename=meshes/link8.STL
Joints:
- removed joint ee_arm
- removed joint ee_bar
- removed joint ee_gripper
- removed joint elbow
- removed joint forearm_roll
- removed joint gripper
- removed joint gripper_bar
- removed joint left_finger
- removed joint right_finger
- removed joint shoulder
- removed joint waist
- removed joint wrist_angle
- removed joint wrist_rotate
- added joint base_to_dummy: type fixed, parent dummy_link, child base_link, origin xyz=0 0 0 rpy=0 0 0
- added joint joint1: type revolute, parent base_link, child link1, origin xyz=0 0 0.123 rpy=0 0 0, axis 0 0 1, limit lower=-2.618 upper=2.168 effort=100 velocity=5
- added joint joint2: type revolute, parent link1, child link2, origin xyz=0 0 0 rpy=1.5708 -0.1359 -3.1416, axis 0 0 1, limit lower=0 upper=3.14 effort=100 velocity=5
- added joint joint3: type revolute, parent link2, child link3, origin xyz=0.28503 0 0 rpy=0 0 -1.7939, axis 0 0 1, limit lower=-2.967 upper=0 effort=100 velocity=5
- added joint joint4: type revolute, parent link3, child link4, origin xyz=-0.021984 -0.25075 0 rpy=1.5708 0 0, axis 0 0 1, limit lower=-1.745 upper=1.745 effort=100 velocity=5
- added joint joint5: type revolute, parent link4, child link5, origin xyz=0 0 0 rpy=-1.5708 0 0, axis 0 0 1, limit lower=-1.22 upper=1.22 effort=100 velocity=5
- added joint joint6: type revolute, parent link5, child link6, origin xyz=8.8259E-05 -0.091 0 rpy=1.5708 0 0, axis 0 0 1, limit lower=-2.0944 upper=2.0944 effort=100 velocity=3
- added joint joint6_to_gripper_base: type fixed, parent link6, child gripper_base, origin xyz=0 0 0 rpy=0 0 0
- added joint joint7: type prismatic, parent gripper_base, child link7, origin xyz=0 0 0.1358 rpy=1.5708 0 0, axis 0 0 1, limit lower=0 upper=0.035 effort=10 velocity=1
- added joint joint8: type prismatic, parent gripper_base, child link8, origin xyz=0 0 0.1358 rpy=1.5708 0 -3.1416, axis 0 0 -1, limit lower=-0.035 upper=0 effort=10 velocity=1
